File: EDA/Pi5CanAndBuckHat/Pi5CanAndBuckHat.kicad_pcb (KiCad board)
At the start: 2 copper layers, 65 x 56.5 mm, 11 parts, among them IC1 MCP2515T-I_SO, IC2 SN65HVD230DR, J1 RPi_GPIO, J2 S4B-XH-SM4-TB, U1 Amazon Buck Converter, Y1 HCM4912000000ABJT

Commit message: Fixing PWA not installing and updated KiCAD EDA files to use library
Parts:
- removed J2: S4B-XH-SM4-TB, Connector_JST:JST_S4B-XH-SM4-TB
- added J3: S4B-XH-SM4-TB, TrailCurrentFootprints:JST_S4B-XH-SM4-TB, F.Cu at (119.0, 82.8)
- C2: footprint easyeda2kicad:C1206 -> Capacitor_SMD:C_1206_3216Metric
- IC1: footprint CustomLibrary:MCP2515T-ISO -> TrailCurrentFootprints:MCP2515T-ISO
- IC2: footprint CustomLibrary:SN65HVD230DR -> TrailCurrentFootprints:SN65HVD230DR
- U1: footprint Converter_DCDC:AmazonBuckConverter -> TrailCurrentFootprints:AmazonBuckConverter
- Y1: footprint CustomLibrary:HCM4912000000ABJT -> TrailCurrentFootprints:HCM4912000000ABJT
Connections:
- C2 pad 1: +3.3V -> unconnected-(C2-Pad1)
- C2 pad 2: GND -> unconnected-(C2-Pad2)
