File: EDA/Pi5CanAndBuckHat/Pi5CanAndBuckHat.kicad_sch (KiCad schematic)
At the start: 11 parts, among them IC1 MCP2515T-I_SO, IC2 SN65HVD230DR, J1 RPi_GPIO, J2 S4B-XH-SM4-TB, U1 Amazon Buck Converter, Y1 HCM4912000000ABJT

Commit message: Fixing PWA not installing and updated KiCAD EDA files to use library
Parts:
- removed J2: S4B-XH-SM4-TB, Connector_JST:JST_S4B-XH-SM4-TB, symbol Connector_Generic:S4B-XH-SM4-TB
- added J3: S4B-XH-SM4-TB, TrailCurrentFootprints:JST_S4B-XH-SM4-TB, symbol TrailCurrentSymbolLibrary:S4B-XH-SM4-TB
- C2: footprint easyeda2kicad:C1206 -> Capacitor_SMD:C_1206_3216Metric; symbol LCSC:CL31B226KPHNNNE -> Device:C; LCSC Part C87996 -> (none)
- IC1: footprint CustomLibrary:MCP2515T-ISO -> TrailCurrentFootprints:MCP2515T-ISO; symbol CustomLibraries:MCP2515T-I_SO -> TrailCurrentSymbolLibrary:MCP2515T-I_SO
- IC2: footprint CustomLibrary:SN65HVD230DR -> TrailCurrentFootprints:SN65HVD230DR; symbol CustomLibraries:SN65HVD230DR -> TrailCurrentSymbolLibrary:SN65HVD230DR
- U1: footprint Converter_DCDC:AmazonBuckConverter -> TrailCurrentFootprints:AmazonBuckConverter
- Y1: footprint CustomLibrary:HCM4912000000ABJT -> TrailCurrentFootprints:HCM4912000000ABJT; symbol CustomLibraries:HCM4912000000ABJT -> TrailCurrentSymbolLibrary:HCM4912000000ABJT
Connections:
- net +12V: now also J3.4
- net +3.3V: no longer C2.1
- net GND: now also J3.3; no longer C2.2
- net PI_CANH: now also J3.2
- net PI_CANL: now also J3.1
